File: example/RPi0PWR/RPi0PWR.brd (EAGLE design)
At the start: 17.8 x 17.8 mm, 6 parts, among them SW1 SW3-1

Commit message: update
Parts:
- removed IN: (no value), jst-ph:JST-PH2
- added BAT: (no value), ytani1:JST-PH2
- DCDC1: value +5V -> (none); device ytani1:DC-DC_5V_0.48A -> ytani1:DCDC-5V-0.48A
- OUT: device jst-ph:JST-PH2 -> ytani1:JST-PH2
- SW1: value SW3-1 -> (none)
Connections:
- removed net +5V: DCDC1.+5V, OUT.2
- removed net BAT+0: IN.2, SW1.1
- new net N$1: DCDC1.+5V, OUT.1
- new net N$2: BAT.1, SW1.1
- net GND: now also BAT.2, OUT.2; no longer IN.1, OUT.1
Routing:
- net N$2: track 0.00 -> 7.89 mm
- net BAT+0: track 7.89 -> 0.00 mm
- net N$1: track 0.00 -> 5.35 mm
- net +5V: track 5.35 -> 0.00 mm
Changed lines of the file:
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@@
 </autorouter>
 <elements>
-<element name="DCDC1" library="ytani1" package="DC-DC_5V_0.48A" value="+5V" x="12.7" y="11.43" smashed="yes" rot="R180">
-<attribute name="URL_AMAZON" value="https://www.amazon.co.jp/gp/product/B07N8TBJB3/" x="-5.08" y="29.21" size="1.778" layer="27" rot="R180" display="off"/>
-</element>
 <element name="LED" library="led" library_urn="urn:adsk.eagle:library:259" package="LED3MM" package3d_urn="urn:adsk.eagle:package:15797/1" value="" x="8.89" y="5.08" smashed="yes">
-<attribute name="NAME" x="6.985" y="0.381" size="1.27" layer="25" ratio="10"/>
+<attribute name="NAME" x="6.985" y="1.651" size="1.27" layer="25" ratio="10"/>
 <attribute name="POPULARITY" value="97" x="36.83" y="-20.32" size="1.778" layer="27" display="off"/>
 <attribute name="VALUE" x="10.795" y="3.429" size="1.27" layer="27" ratio="10"/>
 </element>
-<element name="IN" library="jst-ph" package="JST-PH2" value="" x="3.81" y="2.54" smashed="yes">
-<attribute name="NAME" x="3.35" y="6.0401" size="1.27" layer="25"/>
+<element name="R1" library="rcl" library_urn="urn:adsk.eagle:library:334" package="0204/5" package3d_urn="urn:adsk.eagle:package:23488/1" value="1M" x="7.62" y="10.16" smashed="yes" rot="R90">
+<attribute name="NAME" x="6.35" y="6.35" size="0.9906" layer="25" ratio="10" rot="R90"/>
+<attribute name="POPULARITY" value="18" x="41.91" y="26.67" size="1.778" layer="27" rot="R90" display="off"/>
+<attribute name="SPICEPREFIX" value="R" x="41.91" y="26.67" size="1.778" layer="27" rot="R90" display="off"/>
+<attribute name="VALUE" x="6.35" y="8.89" size="0.9906" layer="27" ratio="10" rot="R90"/>
 </element>
-<element name="OUT" library="jst-ph" package="JST-PH2" value="" x="13.97" y="2.54" smashed="yes" rot="R180">
+<element name="BAT" library="ytani1" package="JST-PH2" value="" x="3.81" y="2.54" smashed="yes">
+<attribute name="NAME" x="0.81" y="6.0401" size="1.27" layer="25"/>
+</element>
+<element name="OUT" library="ytani1" package="JST-PH2" value="" x="13.97" y="2.54" smashed="yes" rot="R180">
 <attribute name="NAME" x="13.51" y="4.7701" size="1.27" layer="25"/>
 </element>
-<element name="R1" library="rcl" library_urn="urn:adsk.eagle:library:334" package="0204/5" package3d_urn="urn:adsk.eagle:package:23488/1" value="1M" x="7.62" y="10.16" smashed="yes" rot="R90">
-<attribute name="NAME" x="6.35" y="7.62" size="0.9906" layer="25" ratio="10" rot="R90"/>
-<attribute name="POPULARITY" value="18" x="41.91" y="26.67" size="1.778" layer="27" rot="R90" display="off"/>
-<attribute name="SPICEPREFIX" value="R" x="41.91" y="26.67" size="1.778" layer="27" rot="R90" display="off"/>
-<attribute name="VALUE" x="6.35" y="10.16" size="0.9906" layer="27" ratio="10" rot="R90"/>
+<element name="SW1" library="ytani1" package="SW3-1" value="" x="2.54" y="12.7" smashed="yes" rot="R90">
+<attribute name="MF" value="HiLetgo" x="2.54" y="12.7" size="1.778" layer="27" rot="R90" display="off"/>
+<attribute name="NAME" x="5.08" y="17.78" size="1.778" layer="21" rot="R270"/>
+<attribute name="URL_AMAZON" value="https://www.amazon.co.jp/gp/product/B01LYVYQNO/" x="2.54" y="12.7" size="1.778" layer="27" rot="R90" display="off"/>
 </element>
-<element name="SW1" library="ytani1" package="SW3-1" value="SW3-1" x="2.54" y="12.7" smashed="yes" rot="R90"/>
+<element name="DCDC1" library="ytani1" package="DCDC-5V-0.48A" value="" x="12.7" y="11.43" smashed="yes" rot="R180">
+<attribute name="URL_AMAZON" value="https://www.amazon.co.jp/gp/product/B07N8TBJB3/" x="12.7" y="11.43" size="1.778" layer="27" rot="R180" display="off"/>
+</element>
 </elements>
 <signals>
 <signal name="GND">
+<contactref element="LED" pad="K"/>
+<wire x1="10.16" y1="2.54" x2="12.7" y2="2.54" width="0.8128" layer="1"/>
+<wire x1="12.7" y1="2.54" x2="12.97" y2="2.54" width="0.8128" layer="1"/>
+<wire x1="10.16" y1="5.08" x2="10.16" y2="2.54" width="0.8128" layer="1"/>
+<contactref element="BAT" pad="2"/>
+<contactref element="OUT" pad="2"/>
+<wire x1="4.81" y1="2.54" x2="10.16" y2="2.54" width="0.8128" layer="1"/>
 <contactref element="DCDC1" pad="GND"/>
-<contactref element="LED" pad="K"/>
-<contactref element="IN" pad="1"/>
-<contactref element="OUT" pad="1"/>
 <wire x1="12.7" y1="7.62" x2="12.7" y2="2.54" width="0.8128" layer="1"/>
-<wire x1="12.7" y1="2.54" x2="12.97" y2="2.54" width="0.8128" layer="1"/>
-<wire x1="4.81" y1="2.54" x2="10.16" y2="2.54" width="0.8128" layer="1"/>
-<wire x1="10.16" y1="2.54" x2="12.7" y2="2.54" width="0.8128" layer="1"/>
-<wire x1="10.16" y1="5.08" x2="10.16" y2="2.54" width="0.8128" layer="1"/>
 </signal>
 <signal name="LED+">
@@
 <signal name="BAT+">
 <contactref element="R1" pad="2"/>
-<contactref element="DCDC1" pad="VIN"/>
-<wire x1="7.62" y1="12.7" x2="10.16" y2="12.7" width="0.8128" layer="1"/>
-<wire x1="10.16" y1="12.7" x2="10.16" y2="7.62" width="0.8128" layer="1"/>
+<wire x1="10.16" y1="12.7" x2="7.62" y2="12.7" width="0.8128" layer="1"/>
+<contactref element="SW1" pad="3"/>
 <contactref element="SW1" pad="2"/>
-<contactref element="SW1" pad="3"/>
 <wire x1="2.54" y1="15.24" x2="2.54" y2="12.7" width="0.8128" layer="1"/>
 <wire x1="2.54" y1="12.7" x2="7.62" y2="12.7" width="0.8128" layer="1"/>
+<contactref element="DCDC1" pad="VIN"/>
+<wire x1="10.16" y1="7.62" x2="10.16" y2="12.7" width="0.8128" layer="1"/>
 </signal>
-<signal name="BAT+0">
-<contactref element="IN" pad="2"/>
-<wire x1="2.54" y1="2.54" x2="2.81" y2="2.54" width="0.8128" layer="1"/>
+<signal name="N$2">
+<contactref element="BAT" pad="1"/>
 <contactref element="SW1" pad="1"/>
-<wire x1="2.54" y1="10.16" x2="2.54" y2="2.54" width="0.8128" layer="1"/>
+<wire x1="2.54" y1="2.54" x2="2.54" y2="10.16" width="0.8128" layer="1"/>
+<wire x1="2.81" y1="2.54" x2="2.54" y2="2.54" width="0.8128" layer="1"/>
 </signal>
-<signal name="+5V">
+<signal name="N$1">
 <contactref element="DCDC1" pad="+5V"/>
-<contactref element="OUT" pad="2"/>
+<contactref element="OUT" pad="1"/>
 <wire x1="15.24" y1="7.62" x2="15.24" y2="2.54" width="0.8128" layer="1"/>
 <wire x1="15.24" y1="2.54" x2="14.97" y2="2.54" width="0.8128" layer="1"/>
