File: example/RPi0PWR/RPi0PWR.sch (EAGLE design)
At the start: 6 parts, among them SW1 SW3-1

Commit message: update
Parts:
- removed IN: (no value), jst-ph:JST-PH2
- added BAT: (no value), ytani1:JST-PH2
- DCDC1: value +5V -> (none); device ytani1:DC-DC_OUT:5V_0.48A -> ytani1:DCDC-5V-0.48A
- OUT: device jst-ph:JST-PH2 -> ytani1:JST-PH2
- SW1: value SW3-1 -> (none)
Connections:
- removed net +5V: DCDC1.VOUT, OUT.2
- removed net BAT+0: IN.2, SW1.1
- new net N$1: DCDC1.VOUT, OUT.1
- new net N$2: BAT.1, SW1.1
- net GND: now also BAT.2, OUT.2; no longer IN.1, OUT.1
Changed lines of the file:
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@@
 </classes>
 <parts>
-<part name="DCDC1" library="ytani1" deviceset="DC-DC_OUT:5V_0.48A" device="" value="+5V"/>
 <part name="GND1" library="supply1" library_urn="urn:adsk.eagle:library:371" deviceset="GND" device=""/>
 <part name="GND2" library="supply1" library_urn="urn:adsk.eagle:library:371" deviceset="GND" device=""/>
 <part name="R1" library="rcl" library_urn="urn:adsk.eagle:library:334" deviceset="R-US_" device="0204/5" package3d_urn="urn:adsk.eagle:package:23488/1" value="1M"/>
 <part name="LED" library="led" library_urn="urn:adsk.eagle:library:259" deviceset="LED" device="3MM" package3d_urn="urn:adsk.eagle:package:15797/1"/>
-<part name="IN" library="jst-ph" deviceset="JST-PH2" device=""/>
-<part name="OUT" library="jst-ph" deviceset="JST-PH2" device=""/>
 <part name="GND3" library="supply1" library_urn="urn:adsk.eagle:library:371" deviceset="GND" device=""/>
 <part name="GND4" library="supply1" library_urn="urn:adsk.eagle:library:371" deviceset="GND" device=""/>
+<part name="FRAME1" library="frames" library_urn="urn:adsk.eagle:library:229" deviceset="A5L-LOC" device=""/>
+<part name="BAT" library="ytani1" deviceset="JST-PH2" device=""/>
+<part name="OUT" library="ytani1" deviceset="JST-PH2" device=""/>
 <part name="SW1" library="ytani1" deviceset="SW3-1" device=""/>
-<part name="FRAME1" library="frames" library_urn="urn:adsk.eagle:library:229" deviceset="A5L-LOC" device=""/>
+<part name="DCDC1" library="ytani1" deviceset="DCDC-5V-0.48A" device=""/>
 </parts>
 <sheets>
@@
 </plain>
 <instances>
-<instance part="DCDC1" gate="G$1" x="43.18" y="33.02" smashed="yes">
-<attribute name="NAME" x="38.1" y="36.83" size="1.778" layer="95"/>
-</instance>
-<instance part="GND1" gate="1" x="17.78" y="7.62" smashed="yes">
-<attribute name="VALUE" x="15.24" y="5.08" size="1.778" layer="96"/>
+<instance part="GND1" gate="1" x="20.32" y="7.62" smashed="yes">
+<attribute name="VALUE" x="17.78" y="5.08" size="1.778" layer="96"/>
 </instance>
 <instance part="GND2" gate="1" x="33.02" y="7.62" smashed="yes">
@@
 <attribute name="VALUE" x="38.735" y="11.938" size="1.778" layer="96" rot="R90"/>
 </instance>
-<instance part="IN" gate="G$1" x="7.62" y="40.64" smashed="yes">
-<attribute name="NAME" x="5.08" y="43.942" size="1.778" layer="95"/>
-<attribute name="VALUE" x="5.08" y="33.274" size="1.778" layer="96"/>
-</instance>
-<instance part="OUT" gate="G$1" x="60.96" y="30.48" smashed="yes" rot="R180">
-<attribute name="NAME" x="55.88" y="36.322" size="1.778" layer="95"/>
-<attribute name="VALUE" x="63.5" y="37.846" size="1.778" layer="96" rot="R180"/>
-</instance>
 <instance part="GND3" gate="1" x="43.18" y="7.62" smashed="yes">
 <attribute name="VALUE" x="40.64" y="5.08" size="1.778" layer="96"/>
@@
 <attribute name="VALUE" x="48.26" y="5.08" size="1.778" layer="96"/>
 </instance>
-<instance part="SW1" gate="G$1" x="25.4" y="33.02" smashed="yes"/>
 <instance part="FRAME1" gate="G$1" x="-58.42" y="-41.91" smashed="yes">
 <attribute name="DRAWING_NAME" x="82.55" y="-26.67" size="2.54" layer="94"/>
 <attribute name="LAST_DATE_TIME" x="82.55" y="-31.75" size="2.286" layer="94"/>
 <attribute name="SHEET" x="95.885" y="-36.83" size="2.54" layer="94"/>
+</instance>
+<instance part="BAT" gate="G$1" x="12.7" y="40.64" smashed="yes" rot="R180">
+<attribute name="NAME" x="17.78" y="37.338" size="1.778" layer="95" rot="R180"/>
+<attribute name="VALUE" x="17.78" y="48.006" size="1.778" layer="96" rot="R180"/>
+</instance>
+<instance part="OUT" gate="G$1" x="58.42" y="33.02" smashed="yes">
+<attribute name="NAME" x="53.34" y="36.322" size="1.778" layer="95"/>
+<attribute name="VALUE" x="53.34" y="25.654" size="1.778" layer="96"/>
+</instance>
+<instance part="SW1" gate="G$1" x="22.86" y="33.02" smashed="yes">
+<attribute name="NAME" x="24.13" y="35.56" size="1.778" layer="95"/>
+</instance>
+<instance part="DCDC1" gate="G$1" x="43.18" y="33.02" smashed="yes">
+<attribute name="NAME" x="38.1" y="36.83" size="1.778" layer="95"/>
 </instance>
 </instances>
@@
 </segment>
 <segment>
-<pinref part="DCDC1" gate="G$1" pin="GND"/>
+<wire x1="15.24" y1="43.18" x2="20.32" y2="43.18" width="0.1524" layer="91"/>
+<pinref part="GND1" gate="1" pin="GND"/>
+<wire x1="20.32" y1="43.18" x2="20.32" y2="10.16" width="0.1524" layer="91"/>
+<pinref part="BAT" gate="G$1" pin="2"/>
+</segment>
+<segment>
+<wire x1="55.88" y1="30.48" x2="50.8" y2="30.48" width="0.1524" layer="91"/>
+<pinref part="GND4" gate="1" pin="GND"/>
+<wire x1="50.8" y1="30.48" x2="50.8" y2="10.16" width="0.1524" layer="91"/>
+<pinref part="OUT" gate="G$1" pin="2"/>
+</segment>
+<segment>
 <pinref part="GND3" gate="1" pin="GND"/>
 <wire x1="43.18" y1="27.94" x2="43.18" y2="10.16" width="0.1524" layer="91"/>
-</segment>
-<segment>
-<pinref part="IN" gate="G$1" pin="1"/>
-<wire x1="15.24" y1="40.64" x2="17.78" y2="40.64" width="0.1524" layer="91"/>
-<pinref part="GND1" gate="1" pin="GND"/>
-<wire x1="17.78" y1="40.64" x2="17.78" y2="10.16" width="0.1524" layer="91"/>
-</segment>
-<segment>
-<pinref part="OUT" gate="G$1" pin="1"/>
-<wire x1="53.34" y1="30.48" x2="50.8" y2="30.48" width="0.1524" layer="91"/>
-<pinref part="GND4" gate="1" pin="GND"/>
-<wire x1="50.8" y1="30.48" x2="50.8" y2="10.16" width="0.1524" layer="91"/>
+<pinref part="DCDC1" gate="G$1" pin="GND"/>
 </segment>
 </net>
@@
 <segment>
 <pinref part="R1" gate="G$1" pin="2"/>
-<wire x1="27.94" y1="33.02" x2="30.48" y2="33.02" width="0.1524" layer="91"/>
 <wire x1="30.48" y1="33.02" x2="33.02" y2="33.02" width="0.1524" layer="91"/>
 <wire x1="33.02" y1="33.02" x2="33.02" y2="30.48" width="0.1524" layer="91"/>
+<wire x1="22.86" y1="25.4" x2="30.48" y2="25.4" width="0.1524" layer="91"/>
+<wire x1="30.48" y1="25.4" x2="30.48" y2="33.02" width="0.1524" layer="91"/>
+<pinref part="SW1" gate="G$1" pin="3"/>
+<wire x1="22.86" y1="27.94" x2="22.86" y2="25.4" width="0.1524" layer="91"/>
+<pinref part="SW1" gate="G$1" pin="2"/>
+<wire x1="27.94" y1="33.02" x2="30.48" y2="33.02" width="0.1524" layer="91"/>
+<junction x="30.48" y="33.02"/>
 <pinref part="DCDC1" gate="G$1" pin="VIN"/>
 <wire x1="35.56" y1="33.02" x2="33.02" y2="33.02" width="0.1524" layer="91"/>
 <junction x="33.02" y="33.02"/>
-<pinref part="SW1" gate="G$1" pin="2"/>
-<pinref part="SW1" gate="G$1" pin="3"/>
-<wire x1="22.86" y1="30.48" x2="22.86" y2="27.94" width="0.1524" layer="91"/>
-<wire x1="22.86" y1="27.94" x2="30.48" y2="27.94" width="0.1524" layer="91"/>
-<wire x1="30.48" y1="27.94" x2="30.48" y2="33.02" width="0.1524" layer="91"/>
-<junction x="30.48" y="33.02"/>
 </segment>
 </net>
-<net name="BAT+0" class="0">
+<net name="N$2" class="0">
 <segment>
-<pinref part="IN" gate="G$1" pin="2"/>
-<wire x1="15.24" y1="38.1" x2="22.86" y2="38.1" width="0.1524" layer="91"/>
+<wire x1="15.24" y1="40.64" x2="22.86" y2="40.64" width="0.1524" layer="91"/>
+<pinref part="BAT" gate="G$1" pin="1"/>
 <pinref part="SW1" gate="G$1" pin="1"/>
-<wire x1="22.86" y1="38.1" x2="22.86" y2="35.56" width="0.1524" layer="91"/>
+<wire x1="22.86" y1="38.1" x2="22.86" y2="40.64" width="0.1524" layer="91"/>
 </segment>
 </net>
-<net name="+5V" class="0">
+<net name="N$1" class="0">
 <segment>
 <pinref part="DCDC1" gate="G$1" pin="VOUT"/>
-<pinref part="OUT" gate="G$1" pin="2"/>
-<wire x1="50.8" y1="33.02" x2="53.34" y2="33.02" width="0.1524" layer="91"/>
+<pinref part="OUT" gate="G$1" pin="1"/>
+<wire x1="50.8" y1="33.02" x2="55.88" y2="33.02" width="0.1524" layer="91"/>
 </segment>
 </net>
